Commit message: updated node and topic configurations

File: ros/src/platypous_gazebo/urdf/platypous.xacro (robot description, xacro)
@@ -22,4 +22,7 @@
     <material name="black">
         <color rgba="${0/255} ${0/255} ${0/255} 1.0"/>
+    </material>
+    <material name="white">
+        <color rgba="${255/255} ${255/255} ${255/255} 1.0"/>
     </material>
 <!-- MACROS -->
@@ -87,5 +90,5 @@
                 <box size="${chassisLength} ${chassisWidth} ${chassisHeight}"/>
             </geometry>
-            <material name="gray"/>
+            <material name="white"/>
         </visual>
         <inertial>
@@ -101,5 +104,5 @@
     </joint>
     <gazebo reference="chassis">
-        <material>Gazebo/Gray</material>
+        <material>Gazebo/White</material>
     </gazebo>
     <!-- wheels -->
@@ -146,22 +149,28 @@
         <visual>
             <geometry>
-                <box size="0.01 0.06 0.02"/>
-            </geometry>
-            <material name="gray"/>
+                <box size="0.03 0.125 0.03"/>
+            </geometry>
+            <material name="black"/>
         </visual>
     </link>
     <joint name="camera_joint" type="fixed">
-        <origin xyz="${(chassisLength / 2) + 0.005} 0 ${chassisHeight / 2}" rpy="0 0 0"/>
-        <parent link="chassis"/>
+        <origin xyz="0.07 0 0.25" rpy="0 0 0"/>
+        <parent link="base_link"/>
         <child link="camera_link"/>
     </joint>
     <gazebo reference="camera_link">
-        <material>Gazebo/Gray</material>
-    </gazebo>
+        <material>Gazebo/Black</material>
+    </gazebo>
+    <link name="camera_optical_frame" />
+    <joint name="camera_optical_joint" type="fixed">
+        <origin xyz="0 0 0" rpy="-1.57 0 -1.57"/>
+        <parent link="camera_link"/>
+        <child link="camera_optical_frame"/>
+    </joint>
     <!-- laser -->
     <link name="laser_link">
         <visual>
             <geometry>
-                <cylinder length="0.02" radius="0.03"/>
+                <cylinder length="0.02" radius="0.034"/>
             </geometry>
             <material name="blue"/>
@@ -169,6 +178,6 @@
     </link>
     <joint name="laser_joint" type="fixed">
-        <origin xyz="0 0 ${chassisHeight / 2 + 0.01}" rpy="0 0 0"/>
-        <parent link="chassis"/>
+        <origin xyz="-0.18 0 0.34" rpy="0 0 0"/>
+        <parent link="base_link"/>
         <child link="laser_link"/>
     </joint>
@@ -187,10 +196,10 @@
             <wheelTorque>${wheelTorque}</wheelTorque>
             <commandTopic>/driver/cmd_vel</commandTopic>
-            <odometryTopic>/differential_drive/odom</odometryTopic>
+            <odometryTopic>/driver/wheel_odometry</odometryTopic>
             <odometryFrame>odom</odometryFrame>
             <robotBaseFrame>base_link</robotBaseFrame>
             <odometrySource>encoder</odometrySource>
-            <publishWheelTF>true</publishWheelTF>
-            <publishOdomTF>false</publishOdomTF>
+            <publishWheelTF>false</publishWheelTF>
+            <publishOdomTF>true</publishOdomTF>
             <publishWheelJointState>false</publishWheelJointState>
             <legacyMode>false</legacyMode>
@@ -224,10 +233,10 @@
                 <alwaysOn>true</alwaysOn>
                 <updateRate>0.0</updateRate>
-                <cameraName>depth_camera</cameraName>
-                <imageTopicName>/depth_camera/color/image_raw</imageTopicName>
-                <cameraInfoTopicName>/depth_camera/color/camera_info</cameraInfoTopicName>
-                <depthImageTopicName>/depth_camera/depth/image_raw</depthImageTopicName>
-                <depthImageInfoTopicName>/depth_camera/depth/camera_info</depthImageInfoTopicName>
-                <pointCloudTopicName>/depth_camera/depth/points</pointCloudTopicName>
+                <cameraName>camera</cameraName>
+                <imageTopicName>/camera/color/image_raw</imageTopicName>
+                <cameraInfoTopicName>/camera/color/camera_info</cameraInfoTopicName>
+                <depthImageTopicName>/camera/aligned_depth_to_color/image_raw</depthImageTopicName>
+                <depthImageInfoTopicName>/camera/aligned_depth_to_color/camera_info</depthImageInfoTopicName>
+                <pointCloudTopicName>/camera/depth/color/points</pointCloudTopicName>
                 <frameName>camera_optical_frame</frameName>
                 <pointCloudCutoff>0.01</pointCloudCutoff>

Commit message: changed robot forward direction and improved navigation params

File: ros/src/platypous_gazebo/urdf/platypous.xacro (robot description, xacro)
@@ -6,5 +6,5 @@
     <xacro:property name="chassisWidth"  value="0.355"  />
     <xacro:property name="chassisMass"   value="8"      />
-    <xacro:property name="chassisOffset" value="-0.170" />
+    <xacro:property name="chassisOffset" value="0.170" />
     <xacro:property name="wheelWidth"    value="0.060" />
     <xacro:property name="wheelRadius"   value="0.055" />
@@ -135,5 +135,5 @@
         <parent link="chassis"/>
         <child link="caster_wheel"/>
-        <origin xyz="${(-chassisLength / 2) + wheelRadius / 2} 0 ${-(wheelRadius + chassisHeight) / 2}" rpy="0 0 0"/>
+        <origin xyz="${(chassisLength / 2) - wheelRadius / 2} 0 ${-(wheelRadius + chassisHeight) / 2}" rpy="0 0 0"/>
     </joint>
     <gazebo reference="caster_wheel">
@@ -155,5 +155,5 @@
     </link>
     <joint name="camera_joint" type="fixed">
-        <origin xyz="0.07 0 0.25" rpy="0 0 0"/>
+        <origin xyz="0.41 0 0.25" rpy="0 0 0"/>
         <parent link="base_link"/>
         <child link="camera_link"/>
@@ -178,5 +178,5 @@
     </link>
     <joint name="laser_joint" type="fixed">
-        <origin xyz="-0.18 0 0.34" rpy="0 0 0"/>
+        <origin xyz="0.18 0 0.34" rpy="0 0 0"/>
         <parent link="base_link"/>
         <child link="laser_link"/>

Commit message: updated robot direction and launch config

File: ros/src/platypous_gazebo/urdf/platypous.xacro (robot description, xacro)
@@ -178,5 +178,5 @@
     </link>
     <joint name="laser_joint" type="fixed">
-        <origin xyz="0.18 0 0.34" rpy="0 0 0"/>
+        <origin xyz="0.18 0 0.34" rpy="0 0 3.141593"/>
         <parent link="base_link"/>
         <child link="laser_link"/>

Commit message: exploration, fixes

File: ros/src/platypous_gazebo/urdf/platypous.xacro (robot description, xacro)
@@ -155,5 +155,5 @@
     </link>
     <joint name="camera_joint" type="fixed">
-        <origin xyz="0.41 0 0.25" rpy="0 0 0"/>
+        <origin xyz="0.0 0 0.6" rpy="0 0 0"/>
         <parent link="base_link"/>
         <child link="camera_link"/>
@@ -188,5 +188,5 @@
     <gazebo>
         <plugin name="differential_drive_controller" filename="libgazebo_ros_diff_drive.so">
-            <updateRate>30</updateRate>
+            <updateRate>100</updateRate>
             <leftJoint>left_wheel_joint</leftJoint>
             <rightJoint>right_wheel_joint</rightJoint>
@@ -216,5 +216,5 @@
     <gazebo reference="camera_link">
         <sensor name="depth_camera" type="depth">
-            <update_rate>30</update_rate>
+            <update_rate>5</update_rate>
             <camera>
                 <horizontal_fov>1.6</horizontal_fov>
@@ -286,3 +286,23 @@
         </sensor>
     </gazebo>
+    <gazebo reference="camera_optical_frame">
+        <gravity>true</gravity>
+        <sensor name="imu_sensor" type="imu">
+            <always_on>true</always_on>
+            <update_rate>200</update_rate>
+            <visualize>true</visualize>
+            <topic>/camera/imu</topic>
+            <plugin filename="libgazebo_ros_imu_sensor.so" name="imu_plugin">
+                <topicName>/camera/imu</topicName>
+                <bodyName>chassis</bodyName>
+                <updateRateHZ>200.0</updateRateHZ>
+                <gaussianNoise>0.01</gaussianNoise>
+                <xyzOffset>0 0 0</xyzOffset>
+                <rpyOffset>0 0 0</rpyOffset>
+                <frameName>camera_optical_frame</frameName>
+                <initialOrientationAsReference>false</initialOrientationAsReference>
+            </plugin>
+            <pose>0 0 0 0 0 0</pose>
+        </sensor>
+    </gazebo>
 </robot>
